File: Flash_ID_Spoofer.kicad_pcb (KiCad board)
At the start: 2 copper layers, 34.9 x 14.4 mm, 4 parts, among them J1 SOIC8-PAD, J2 Conn_01x06, U1 EPM3032ATC44-10_TQFP-44, U2 W25Q128JVS

Commit message: adjust details
Routing:
- net GND: track 55.1 -> 53.1 mm

Commit message: Update for PCB
Other:
- board size 34.9 x 14.4 mm -> 34.9 x 15.5 mm
- board text added: "JLCJLCJLCJLC"
