File: Flash_ID_Spoofer.kicad_pcb (KiCad board)
At the start: 2 copper layers, 34.9 x 15.5 mm, 4 parts, among them J1 SOIC8-PAD, J2 Conn_01x06, U1 EPM3032ATC44-10_TQFP-44, U2 W25Q128JVS

Commit message: add gnd via holes
Routing:
- net GND: vias 8 -> 15

Commit message: Update PCB
Parts:
- moved J2 10.00 mm to (144.7, 103.4), turned to 180 degrees
- turned U1 to 270 degrees
Routing:
- net GND: track 53.1 -> 0.00 mm, vias 15 -> 13
- net /FROM_FLASH: track 17.0 -> 3.32 mm, vias 2 -> 0
- net /FROM_CPU: track 30.5 -> 17.0 mm, vias 4 -> 0
- net /TO_CPU: track 30.7 -> 18.3 mm
- net /CS: track 32.2 -> 21.3 mm, vias 3 -> 1
- net /SCLK: track 29.0 -> 18.1 mm, vias 2 -> 0
- net /TDI: track 9.78 -> 17.3 mm
- net /TDO: track 9.50 -> 15.0 mm, vias 0 -> 1
- net /WP: track 19.2 -> 13.9 mm, vias 2 -> 1
- net /TCK: track 13.0 -> 9.82 mm
- net VCC: track 49.0 -> 52.0 mm
- net /TMS: track 12.8 -> 11.6 mm
- net /HOLD: track 7.14 -> 7.72 mm
Other:
- board size 34.9 x 15.5 mm -> 34.9 x 15.1 mm
